File: PCB/Chest/Chest.kicad_pcb (KiCad board)
At the start: 2 copper layers, 70 x 70 mm, 47 parts, among them J1 Reset, J2 LED, J3 TC2030-USB-NL-DS, J4 SPK, J5 USB-C-Socket-H, J6 Power, SW1 Button, U1 ICS43434_MEMS_Mic, U2 MAX98357A, U3 Relay, U5 IRM-H638T/TR2, U6 ESP32-S3-MINI-1, U7 MD8942, U8 VEML6040

Commit message: Started Chest board
Parts:
- removed JP1: PWR, RevK:Pad_1206_0805_Bridged
- removed L2: 10uH, RevK:L_4x4_
- removed SW1: Button, RevK:SW_Push_1P1T_NO_6x6mm
- removed U7: MD8942, RevK:SOT-23-6-MD8942
- removed U8: VEML6040, RevK:VEML6040
- added C6: 22uF 35V, RevK:C_1210, F.Cu at (111.0, 91.5)
- added D4: ~, RevK:DFN1006-2L, F.Cu at (88.4, 95.5)
- added D5: ~, RevK:DFN1006-2L, F.Cu at (112.5, 95.5)
- added D6: ~, RevK:DFN1006-2L, F.Cu at (88.0, 102.0)
- added D7: ~, RevK:DFN1006-2L, F.Cu at (111.5, 106.5)
- added J10: L, RevK:WAGO-2060-452-998-404, F.Cu at (80.0, 85.0)
- added J11: R, RevK:WAGO-2060-452-998-404, F.Cu at (120.0, 85.0)
- added J12: TF_PUSH, RevK:TF_PUSH, F.Cu at (104.8, 115.0)
- added J7: 2, RevK:WAGO-2060-453-998-404, F.Cu at (120.0, 95.5)
- added J8: 3, RevK:WAGO-2060-453-998-404, F.Cu at (80.0, 108.0)
- added J9: 4, RevK:WAGO-2060-453-998-404, F.Cu at (120.0, 108.0)
- added L1: 10uH, RevK:L_4x4_, F.Cu at (94.0, 106.5)
- added R10: 10K, RevK:R_0402, F.Cu at (99.5, 105.0)
- added R11: 10K, RevK:R_0402, F.Cu at (100.5, 105.0)
- added R12: 10K, RevK:R_0402, F.Cu at (102.5, 105.0)
- added R13: 10K, RevK:R_0402, F.Cu at (105.0, 105.0)
- added R16: 210R2, RevK:R_0402, F.Cu at (108.5, 87.5)
- added U4: R, RevK:ICS43434_MEMS_Mic_Open, F.Cu at (111.0, 83.0)
- added V3: ~, RevK:VCUT70N, F.Cu at (128.0, 100.0)
- added V4: ~, RevK:VCUT70N, F.Cu at (72.5, 100.0)
- C1: value 220uF Tant -> 10uF 35V; footprint RevK:CP_EIA-3528-21_Kemet-B -> RevK:C_0603_
- C10: value 10uF 35V -> 100nF; footprint RevK:C_0603_ -> RevK:C_0402
- C11: value 10uF 6.3V -> 10uF; footprint RevK:C_0603_ -> RevK:C_0402
- C12: value 100nF -> 10uF; footprint RevK:C_0603_ -> RevK:C_0402
- C13: value 10uF -> 100nF
- C2: value 100nF -> 10uF 6.3V; footprint RevK:C_0402 -> RevK:C_0603_
- C3: value 22uF -> 100nF; footprint RevK:C_0603 -> RevK:C_0603_
- C4: value 4.7uF -> 1uF
- C5: value 10uF 35V -> 22uF 35V; footprint RevK:C_0603 -> RevK:C_1210
- C7, C8: value 10uF -> 22uF 35V; footprint RevK:C_0402 -> RevK:C_1210
- C9: value 1uF -> 100nF
- D1: value XL-1010RGBC-WS2812B -> ~; footprint RevK:SMD1010 -> RevK:DFN1006-2L
- D3: value ~ -> XL-1010RGBC-WS2812B; footprint RevK:DFN1006-2L -> RevK:SMD1010
- J2: value LED -> A; footprint RevK:WAGO-2060-453-998-404 -> RevK:WAGO-2060-452-998-404
- J3: value TC2030-USB-NL-DS -> B; footprint RevK:Tag-Connect_TC2030-IDC-NL_2x03_P1.27mm_Vertical -> RevK:WAGO-2060-452-998-404; moved to F.Cu
- J4: value SPK -> TC2030-USB-NL-DS; footprint RevK:WAGO-2060-452-998-404 -> RevK:Tag-Connect_TC2030-IDC-NL_2x03_P1.27mm_Vertical
- J6: value Power -> 1; footprint RevK:WAGO-2060-452-998-404 -> RevK:WAGO-2060-453-998-404
- R1: value 124K -> 124k; footprint RevK:R_0402 -> RevK:R_0402_
- R14: value 39k2 -> 10K; footprint RevK:R_0402_ -> RevK:R_0402
- R15: value 1M -> 10K; footprint RevK:R_0402_ -> RevK:R_0402
- R2: value 10K -> 39k2; footprint RevK:R_0402 -> RevK:R_0402_
- R3: value 10K -> 1M; footprint RevK:R_0402 -> RevK:R_0402_
- R4: value 124k -> 10K; footprint RevK:R_0402_ -> RevK:R_0402
- R5, R6: value 5K1 -> 10K
- R7: value 1K -> 5K1
- R8: value 634K -> 5K1
- R9: value 100R -> 10K
- U1: value ICS43434_MEMS_Mic -> MD8942; footprint RevK:ICS43434_MEMS_Mic_Open -> RevK:SOT-23-6-MD8942
- U2: value MAX98357A -> ESP32-S3-MINI-1; footprint RevK:WLP-1.437mmx1.347mm-0.21mm-ball -> RevK:ESP32-S3-MINI-1
- U3: value Relay -> L; footprint RevK:SO-4_4.4x4.3mm_P2.54mm -> RevK:ICS43434_MEMS_Mic_Open
- U5: value IRM-H638T/TR2 -> MAX98357A; footprint RevK:SMD-4P,4x5mm -> RevK:WLP-1.437mmx1.347mm-0.21mm-ball
- U6: value ESP32-S3-MINI-1 -> MAX98357A; footprint RevK:ESP32-S3-MINI-1 -> RevK:WLP-1.437mmx1.347mm-0.21mm-ball
- moved U1 33.8 mm to (89.5, 106.5), turned to 90 degrees
- moved R8 31.5 mm to (95.5, 112.0)
- moved D2 31.4 mm to (113.0, 112.5), turned to 90 degrees
- moved J5 30.8 mm to (91.5, 117.0), turned to 0 degrees
- moved J2 29.9 mm to (80.0, 118.5)
- moved U5 27.9 mm to (89.3, 88.0)
- moved C1 27.1 mm to (90.8, 109.0)
- moved C14 26.9 mm to (91.5, 90.0), turned to 90 degrees
- moved R4 26.0 mm to (95.5, 113.5)
- moved C13 25.3 mm to (91.5, 92.0)
- moved C5 24.9 mm to (89.0, 99.5)
- moved D3 24.0 mm to (109.6, 94.4)
- moved J3 22.5 mm to (120.0, 118.5)
- moved R6 21.1 mm to (108.5, 89.5)
- moved C2 20.8 mm to (90.8, 104.0), turned to 180 degrees
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Connections:
- C4 pad 1: Net-(U5-VCC) -> Net-(U2-EN)
- C5 pad 1: DC -> GND
- C5 pad 2: GND -> DC
- C7 pad 1: +3V3 -> GND
- C7 pad 2: GND -> DC
- C8 pad 1: +3V3 -> GND
- C8 pad 2: GND -> DC
- C9 pad 1: Net-(U6-EN) -> GND
- C9 pad 2: GND -> +3V3
- D1 pad 1: unconnected-(D1-O-Pad1) -> BTNA
- D1 pad 2: +3V3 -> GND
- D2 pad 1: GND -> BTNB
- D2 pad 2: LED2 -> GND
- D3 pad 1: GND -> unconnected-(D3-O-Pad1)
- D3 pad 2: PUSH -> +3V3
- J2 pad 2: LED2 -> BTNA
- J3 pad 1: DC -> GND
- J3 pad 2: DC -> BTNB
- J4 pad 1: Net-(J4-Pin_1) -> DC
- J4 pad 2: Net-(J4-Pin_2) -> DC
- J6 pad 2: Net-(J6-Pin_2) -> LED1
- R5 pad 1: Net-(J5-CC1) -> BTNB
- R5 pad 2: GND -> +3V3
- R6 pad 1: GND -> +3V3
- R6 pad 2: Net-(J5-CC2) -> Net-(U2-EN)
- R7 pad 1: Net-(R7-Pad1) -> Net-(J5-CC1)
- R7 pad 2: RELAY -> GND
- R8 pad 1: Net-(U2-~{SD_MODE}) -> GND
- R8 pad 2: SKPPWR -> Net-(J5-CC2)
- R9 pad 1: Net-(U5-VCC) -> +3V3
- R9 pad 2: +3V3 -> SDCD
- U1 pad 1: MICWS -> unconnected-(U1-Pad1)_1
- U1 pad 3: GND -> unconnected-(U1-Pad3)
- U1 pad 4: MICSCK -> unconnected-(U1-EN-Pad4)
- U1 pad 5: +3V3 -> DC
- U1 pad 6: MICSD -> unconnected-(U1-Pad6)
- U3 pad 1: Net-(R7-Pad1) -> MICWS
- U3 pad 3: Net-(J2-Pin_3) -> GND
- U3 pad 4: Net-(J6-Pin_2) -> MICSCK
Routing:
- net DC: track 120.4 -> 0.00 mm, vias 7 -> 0
- net GND: track 84.0 -> 0.00 mm, vias 42 -> 0
- net +3V3: track 79.8 -> 0.00 mm, vias 3 -> 0
- net D-: track 29.8 -> 0.00 mm, vias 2 -> 0
- net LED2: track 27.7 -> 0.00 mm, vias 3 -> 0
- net SKPSD: track 27.3 -> 0.00 mm, vias 2 -> 0
- net SKPSCK: track 26.7 -> 0.00 mm, vias 2 -> 0
- net SKPWS: track 24.6 -> 0.00 mm, vias 2 -> 0
- net Net-(J6-Pin_2): track 24.3 -> 0.00 mm, vias 1 -> 0
- net Net-(J4-Pin_2): track 23.4 -> 0.00 mm, vias 2 -> 0
- net D+: track 23.1 -> 0.00 mm, vias 2 -> 0
- net SKPPWR: track 22.8 -> 0.00 mm, vias 2 -> 0
- net MICSCK: track 22.0 -> 0.00 mm, vias 2 -> 0
- net Net-(U6-EN): track 21.8 -> 0.00 mm, vias 2 -> 0
- net PUSH: track 21.3 -> 0.00 mm, vias 2 -> 0
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- removed copper zone on F.Cu, net DC
Other:
- board text removed: "${CURRENT_DATE}"
- board text removed: "(5V WHEN USB)"
- board text removed: "+"
- board text removed: "-"
- board text removed: "11"
- board text removed: "12"
- board text removed: "13"
- board text removed: "21"
- board text removed: "4"
- board text removed: "44"
- board text removed: "48"
- board text removed: "4V-35V POWER"
- board text removed: "4Ω"
- board text removed: "5V- 35V"
- board text removed: "6x6 BTN"
- board text removed: "8"
- board text removed: "A"
- board text removed: "ADC"
- board text removed: "C2"
- board text removed: "C42"
- board text removed: "C47D33"
- board text removed: "D3"
- board text removed: "D41"
- board text removed: "EXTERNAL"
- board text removed: "HomeIsWhereTheSmartIs"
- board text removed: "I/O 3.3V"
- board text removed: "I2S"
- board text removed: "IR 38kHz"
- board text removed: "L"
- board text removed: "L+R"
- board text removed: "LED"
- board text removed: "Made by RevK www.me.uk"
- board text removed: "Made in China"
- board text removed: "SWITCHED"
- board text removed: "U"
- board text removed: "USB"
- board text removed: "USB 5V"
- board text removed: "USB ONLY IF NOT EXTERNAL POWER"
- board text removed: "W1"
- board text removed: "W40"
- board text removed: "led.revk.uk"
- board text removed: "®"
- board text removed: "⎍"
