File: PCB/Chest/Chest.kicad_pcb (KiCad board)
At the start: 2 copper layers, 70 x 70 mm, 62 parts, among them J1 Reset, J10 L, J11 R, J12 TF_PUSH, J2 A, J3 B, J4 TC2030-USB-NL-DS, J5 USB-C-Socket-H, J6 1, J7 2, J8 3, J9 4, U1 MD8942, U2 ESP32-S3-MINI-1, U3 L, U4 R, U5 MAX98357A, U6 MAX98357A

Commit message: Bigger caps
Parts:
- added C15: 100nF, RevK:C_0402, F.Cu at (91.0, 92.5)
- added C16: 22uF, RevK:C_0603, F.Cu at (91.0, 90.0)
- C5, C6, C7, C8: value 22uF 35V -> C_Polarized; footprint RevK:C_1210 -> RevK:CP_EIA-7343-31_Kemet-D
- moved C11 26.3 mm to (86.0, 90.0), turned to 180 degrees
- moved C14 20.5 mm to (112.0, 90.0), turned to 180 degrees
- moved J4 19.6 mm to (90.5, 101.0)
- moved D3 19.2 mm to (90.5, 96.5)
- moved R4 13.0 mm to (84.5, 120.5), turned to -90 degrees
- moved D1 10.3 mm to (84.5, 118.5), turned to 90 degrees
- moved R8 9.62 mm to (86.0, 113.5), turned to -90 degrees
- moved R2 9.38 mm to (90.2, 113.7), turned to 180 degrees
- moved R7 8.63 mm to (85.0, 113.5), turned to 90 degrees
- moved R1 8.46 mm to (92.0, 113.7), turned to 180 degrees
- moved R3 8.26 mm to (93.8, 113.7), turned to 180 degrees
- moved R16 7.91 mm to (115.0, 83.0)
- moved C2 6.62 mm to (89.5, 110.5), turned to -90 degrees
- moved D2 6.50 mm to (115.5, 118.5), turned to -90 degrees
- moved U1 5.88 mm to (92.0, 111.8), turned to 180 degrees
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Connections:
- C5 pad 1: GND -> DC
- C5 pad 2: DC -> GND
- C6 pad 1: GND -> DC
- C6 pad 2: DC -> GND
- C7 pad 1: GND -> DC
- C7 pad 2: DC -> GND
- C8 pad 1: GND -> DC
- C8 pad 2: DC -> GND
- U2 pad 10: unconnected-(U2-GPIO6-Pad10) -> LED1
- U2 pad 11: LED0 -> LED3
- U2 pad 12: LED1 -> unconnected-(U2-GPIO8-Pad12)
- U2 pad 13: LED2 -> unconnected-(U2-GPIO9-Pad13)
- U2 pad 14: LED3 -> unconnected-(U2-GPIO10-Pad14)
- U2 pad 15: LED4 -> unconnected-(U2-GPIO11-Pad15)
- U2 pad 16: SDDAT2 -> BTNA
- U2 pad 17: SDDAT3 -> BTNB
- U2 pad 18: SDCMD -> unconnected-(U2-GPIO14-Pad18)
- U2 pad 19: SDCLK -> unconnected-(U2-GPIO15-Pad19)
- U2 pad 20: SDDAT0 -> unconnected-(U2-GPIO16-Pad20)
- U2 pad 21: SDDAT1 -> unconnected-(U2-GPIO17-Pad21)
- U2 pad 22: SDCD -> unconnected-(U2-GPIO18-Pad22)
- U2 pad 27: unconnected-(U2-GPIO47-Pad27) -> SDCD
- U2 pad 28: BTNA -> SDDAT1
- U2 pad 29: BTNB -> SDDAT0
- U2 pad 31: unconnected-(U2-GPIO35-Pad31) -> SDCLK
- U2 pad 32: unconnected-(U2-GPIO36-Pad32) -> SDCMD
- U2 pad 33: unconnected-(U2-GPIO37-Pad33) -> SDDAT3
- U2 pad 34: unconnected-(U2-GPIO38-Pad34) -> SDDAT2
- U2 pad 36: MICWS -> unconnected-(U2-GPIO40-Pad36)
- U2 pad 37: MICSD -> LED4
- U2 pad 38: MICSCK -> LED2
- U2 pad 39: unconnected-(U2-GPIO43-Pad39) -> MICSD
- U2 pad 40: SPKPWR -> MICSCK
- U2 pad 44: unconnected-(U2-GPIO46-Pad44) -> MICWS
- U2 pad 8: LED2 -> SPKPWR
- U2 pad 9: unconnected-(U2-GPIO5-Pad9) -> LED0

Commit message: Tracked
Parts:
- moved R16 8.63 mm to (110.1, 90.1)
- moved C12 4.60 mm to (113.8, 85.4)
- moved C14 4.60 mm to (111.8, 85.4)
- moved D4 2.34 mm to (89.8, 96.7)
- moved C13 2.24 mm to (86.0, 89.0), turned to 180 degrees
- moved D5 1.50 mm to (110.5, 97.0)
- moved C10 0.90 mm to (111.0, 83.9), turned to -90 degrees
- moved D3 0.70 mm to (91.2, 96.5)
- moved C9 0.41 mm to (84.6, 82.4)
- turned C6 to -90 degrees
Connections:
- C15 pad 1: +3.3V -> +3V3
- C16 pad 1: +3.3V -> +3V3
- U2 pad 39: MICSD -> MICSCK
- U2 pad 40: MICSCK -> MICSD
Routing:
- net +3V3: track 0.00 -> 207.4 mm, vias 0 -> 7
- net DC: track 0.00 -> 156.0 mm, vias 0 -> 5
- net GND: track 0.00 -> 51.4 mm, vias 0 -> 28
- net MICSD: track 0.00 -> 49.2 mm, vias 0 -> 3
- net MICSCK: track 0.00 -> 47.8 mm, vias 0 -> 3
- net SPKWS: track 0.00 -> 46.5 mm, vias 0 -> 3
- net SPKSD: track 0.00 -> 46.1 mm, vias 0 -> 3
- net SPKSCK: track 0.00 -> 45.2 mm, vias 0 -> 3
- net MICWS: track 0.00 -> 44.5 mm, vias 0 -> 3
- net BTNB: track 0.00 -> 44.1 mm, vias 0 -> 2
- net D+: track 0.00 -> 42.9 mm, vias 0 -> 3
- net BTNA: track 0.00 -> 40.9 mm, vias 0 -> 2
- net SPKPWR: track 0.00 -> 37.4 mm, vias 0 -> 3
- net LED3: track 0.00 -> 33.9 mm, vias 0 -> 2
- net D-: track 0.00 -> 33.8 mm, vias 0 -> 3
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Other:
- board text added: "${CURRENT_DATE}"
- board text added: "+"
- board text added: "-"
- board text added: "1 2 3 4"
- board text added: "12"
- board text added: "13"
- board text added: "21"
- board text added: "38 37 36 35 34 33 47"
- board text added: "41"
- board text added: "42"
- board text added: "43 46 44"
- board text added: "4Ω"
- board text added: "5"
- board text added: "6"
- board text added: "7"
- board text added: "BTN"
- board text added: "DAT2 DAT3 CMD CLK DAT0 DAT1 CD"
- board text added: "L"
- board text added: "LED"
- board text added: "MIC"
- board text added: "Made in China for Andrews&Arnold Ltd"
- board text added: "R"
- board text added: "SCK WS SD"
- board text added: "SD"
- board text added: "SPK"
- board text added: "WS SCK SD PWR"
- board text added: "ironman.revk.uk hiwtsi.uk"

Commit message: Tidy
Parts:
- removed V1, V4: ~, RevK:VCUT70N
- moved V3 35.9 mm to (100.0, 81.0), turned to 0 degrees
- moved R7 1.00 mm to (86.0, 113.5)
- moved R8 1.00 mm to (85.0, 113.5)
- moved V2 0.50 mm to (100.0, 123.0)
Routing:
- net GND: track 51.4 -> 111.0 mm, vias 28 -> 31
- net LED3: track 33.9 -> 36.6 mm
- net SPKPWR: track 37.4 -> 36.0 mm
- net Net-(J5-CC1): track 7.89 -> 8.49 mm
Other:
- board text added: "Designed by RevK www.me.uk"
- board text added: "MicroSD"
- board text removed: "SD"

Commit message: Tweak tracks
Parts:
- R16: value 210R2 -> 210R
Routing:
- net BTNA: track 40.6 -> 44.1 mm
- net DC: track 155.9 -> 152.6 mm
- net D+: track 42.9 -> 46.2 mm
- net +3V3: track 206.9 -> 209.1 mm
- net D-: track 33.8 -> 35.7 mm
- net BTNB: track 44.1 -> 44.7 mm
- net GND: vias 31 -> 39
- added copper zone on F.Cu, net DC

Commit message: New render
Parts:
- removed REF**: Shadow, RevK:Shadow
Other:
- copper layers 2 -> 4
