File: PCB/Chest/Chest.kicad_sch (KiCad schematic)
At the start: 35 parts, among them J1 Reset, J2 TF_PUSH, J3 TC2030-USB-NL-DS, J4 SPK, J5 USB-C-Socket-H, J7 SPK, U1 MAX98357A, U2 ESP32-S3-MINI-1, U2 MAX98357A, U5 MD8942

Commit message: Started Chest board
Parts:
- removed C4: 10uF, RevK:C_0402, symbol Device:C
- added C10, C13, C9: 100nF, RevK:C_0402, symbol Device:C
- added C11: 10uF, RevK:C_0402, symbol Device:C
- added C5, C7, C8: 22uF 35V, RevK:C_1210, symbol Device:C
- added D1, D2, D4, D5, D6, D7: ~, RevK:DFN1006-2L, symbol RevK:ES05D1MC10
- added D3: XL-1010RGBC-WS2812B, RevK:SMD1010, symbol RevK:WS2812B-1mm
- added J2: A, RevK:WAGO-2060-452-998-404, symbol Connector_Generic:Conn_01x02
- added J3: B, RevK:WAGO-2060-452-998-404, symbol Connector_Generic:Conn_01x02
- added J6: 1, RevK:WAGO-2060-453-998-404, symbol Connector_Generic:Conn_01x03
- added J7: 2, RevK:WAGO-2060-453-998-404, symbol Connector_Generic:Conn_01x03
- added J8: 3, RevK:WAGO-2060-453-998-404, symbol Connector_Generic:Conn_01x03
- added J9: 4, RevK:WAGO-2060-453-998-404, symbol Connector_Generic:Conn_01x03
- added R16: 210R2, RevK:R_0402, symbol Device:R
- added R4, R5: 10K, RevK:R_0402, symbol Device:R
- added U3: L, RevK:ICS43434_MEMS_Mic_Open, symbol RevK:ICS43434_MEMS_Mic
- added U4: R, RevK:ICS43434_MEMS_Mic_Open, symbol RevK:ICS43434_MEMS_Mic
- added V3, V4: ~, RevK:VCUT70N, symbol RevK:VCUT
- C6: value 100nF -> 22uF 35V; footprint RevK:C_0402 -> RevK:C_1210
- J10: renamed from J7; value SPK -> L
- J11: renamed from J4; value SPK -> R
- renumbered C13 to C12, J2 to J12, J3 to J4, R3 to R10, R7 to R11, R8 to R12, R9 to R13, R10 to R14, R11 to R15, R5 to R7, R6 to R8, R1 to R9, U1 to U5, U2 to U6
Connections:
- net ADC is gone; now on net SDDAT3: U2.17 (GPIO13)
- net RELAY is gone; now on net SDDAT2: U2.16 (GPIO12)
- net SKPPWR is gone; now on net SPKPWR: U2.40 (GPIO44)
- net +3V3: now also C10.2, C11.1, C13.1, C9.2, D3.2 (+), R4.2, R5.2, U3.5 (VDD), U4.2 (LR), U4.5 (VDD); no longer C6.1
- net DC: now also C6.2, C5.2, C7.2, C8.2, J6.3 (Pin_3), J7.3 (Pin_3), J8.3 (Pin_3), J9.3 (Pin_3)
- net GND: now also C6.1, U5.B2 (GAIN_SLOT), U6.B2 (GAIN_SLOT), C10.1, C11.2, C13.2, C5.1, C7.1, C8.1, C9.1, D1.2, D2.2, D3.3 (-), D4.2, D5.2, D6.2, D7.2, J2.1 (Pin_1), J3.1 (Pin_1), J6.1 (Pin_1), J7.1 (Pin_1), J8.1 (Pin_1), J9.1 (Pin_1), U3.2 (LR), U3.3 (GND), U4.3 (GND); no longer C6.2
- net LED1: now also D4.1, J6.2 (Pin_2)
- net LED2: now also U2.13 (GPIO9), D5.1, J7.2 (Pin_2)
- net MICSCK: now also U3.4 (SCK), U4.4 (SCK)
- net MICSD: now also U3.6 (SD), U4.6 (SD)
- net MICWS: now also U3.1 (WS), U4.1 (WS)
- net SDCD: now also U2.22 (GPIO18)
- net SDCLK: now also U2.19 (GPIO15)
- net SDCMD: now also U2.18 (GPIO14)
- net SDDAT0: now also U2.20 (GPIO16)
- net SDDAT1: now also U2.21 (GPIO17)
- net LED0: now reaches U2.11 (GPIO7)
- net LED0: now also D3.4 (I)
- net LED3: now reaches U2.14 (GPIO10)
- net LED3: now also D6.1, J8.2 (Pin_2)
- net BTNB: now reaches U2.29 (GPIO34)
- net BTNB: now also D2.1, J3.2 (Pin_2), R5.1
- net SPKPWR: now reaches U5.A1 (~{SD_MODE})
- net SPKPWR: now also R16.2
- net at U6.A1 (~{SD_MODE}): now also R16.1
- net IR: no longer names the net of U2.30 (GPIO48)
- net PUSH renamed LED4
- net LED4: now also D7.1, J9.2 (Pin_2)
- net SCL: no longer names the net of U2.27 (GPIO47)
- net SDA renamed BTNA
- net BTNA: now also D1.1, J2.2 (Pin_2), R4.1
- net SKPSCK renamed SPKSCK
- net SKPSD renamed SPKSD
- net SKPWS renamed SPKWS
- no-connect marks 21 -> 15
Other:
- note removed: "SD card multiple inputs multiple LED speakers as L and R"
- moved on the sheet: C12, C6, C7, C8, J12, J4, J5, L2, R10, R11, R12, R13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

Commit message: Tidy
Other:
- title: LED driver -> IronMan Chest
Changed lines of the file:
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@@
 	(paper "A4")
 	(title_block
-		(title "LED driver")
+		(title "IronMan Chest")
 		(rev "1")
 		(comment 1 "@TheRealRevK")

Commit message: Bigger caps
Parts:
- removed C5, C6, C7, C8: 22uF 35V, RevK:C_1210, symbol Device:C
- added C15: 100nF, RevK:C_0402, symbol Device:C
- added C16: 22uF, RevK:C_0603, symbol Device:C
- added C5, C6, C7, C8: C_Polarized, RevK:CP_EIA-7343-31_Kemet-D, symbol Device:C_Polarized
- renumbered V4 to V1, V1 to V2, V2 to V3, V3 to V4
Connections:
- net BTNA: now also U2.16 (GPIO12); no longer U2.28 (GPIO33)
- net BTNB: now also U2.17 (GPIO13); no longer U2.29 (GPIO34)
- net DC: now also C5.1, C6.1, C7.1, C8.1
- net GND: now also C15.2, C16.2, C5.2, C6.2, C7.2, C8.2
- net LED0: now also U2.9 (GPIO5); no longer U2.11 (GPIO7)
- net LED1: now also U2.10 (GPIO6); no longer U2.12 (GPIO8)
- net LED2: now also U2.38 (GPIO42); no longer U2.13 (GPIO9), U2.8 (GPIO4)
- net LED3: now also U2.11 (GPIO7); no longer U2.14 (GPIO10)
- net LED4: now also U2.37 (GPIO41); no longer U2.15 (GPIO11)
- net MICSCK: now also U2.40 (GPIO44); no longer U2.38 (GPIO42)
- net MICSD: now also U2.39 (GPIO43); no longer U2.37 (GPIO41)
- net MICWS: now also U2.44 (GPIO46); no longer U2.36 (GPIO40)
- net SDCD: now also U2.27 (GPIO47); no longer U2.22 (GPIO18)
- net SDCLK: now also U2.31 (GPIO35); no longer U2.19 (GPIO15)
- net SDCMD: now also U2.32 (GPIO36); no longer U2.18 (GPIO14)
- net SDDAT0: now also U2.29 (GPIO34); no longer U2.20 (GPIO16)
- net SDDAT1: now also U2.28 (GPIO33); no longer U2.21 (GPIO17)
- net SDDAT2: now also U2.34 (GPIO38); no longer U2.16 (GPIO12)
- net SDDAT3: now also U2.33 (GPIO37); no longer U2.17 (GPIO13)
- net SPKPWR: now also U2.8 (GPIO4); no longer U2.40 (GPIO44)
- new net +3.3V: C15.1, C16.1
- no-connect marks 15 -> 16
Other:
- moved on the sheet: J6, J7, J8, J9

Commit message: Tracked
Connections:
- net +3.3V is gone; now on net +3V3: C15.1, C16.1
- net MICSCK: now also U2.39 (GPIO43); no longer U2.40 (GPIO44)
- net MICSD: now also U2.40 (GPIO44); no longer U2.39 (GPIO43)
Changed lines of the file:
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@@
 	(global_label "MICSCK"
 		(shape output)
-		(at 66.04 53.34 0)
+		(at 66.04 50.8 0)
 		(fields_autoplaced yes)
 		(effects
@@
 		)
 		(property "Intersheetrefs" "${INTERSHEET_REFS}"
-			(at 75.4467 53.34 0)
+			(at 75.4467 50.8 0)
 			(effects
 				(font
@@
 	(global_label "MICSD"
 		(shape input)
-		(at 66.04 50.8 0)
+		(at 66.04 53.34 0)
 		(fields_autoplaced yes)
 		(effects
@@
 		)
 		(property "Intersheetrefs" "${INTERSHEET_REFS}"
-			(at 74.1767 50.8 0)
+			(at 74.1767 53.34 0)
 			(effects
 				(font
@@
 	)
 	(symbol
+		(lib_id "power:+3.3V")
+		(at 34.29 114.935 0)
+		(unit 1)
+		(exclude_from_sim no)
+		(in_bom yes)
+		(on_board yes)
+		(dnp no)
+		(fields_autoplaced yes)
+		(property "Reference" "#PWR054"
+			(at 34.29 118.745 0)
+			(effects
+				(font
+					(size 1.27 1.27)
+				)
+				(hide yes)
+			)
+		)
+		(property "Value" "+3V3"
+			(at 34.29 111.3592 0)
+			(effects
+				(font
+					(size 1.27 1.27)
+				)
+			)
+		)
+		(property "Footprint" ""
+			(at 34.29 114.935 0)
+			(effects
+				(font
+					(size 1.27 1.27)
+				)
+				(hide yes)
+			)
+		)
+		(property "Datasheet" ""
+			(at 34.29 114.935 0)
+			(effects
+				(font
+					(size 1.27 1.27)
+				)
+				(hide yes)
+			)
+		)
+		(property "Description" "Power symbol creates a global label with name \"+3.3V\""
+			(at 34.29 114.935 0)
+			(effects
+				(font
+					(size 1.27 1.27)
+				)
+				(hide yes)
+			)
+		)
+		(pin "1"
+		)
+		(instances
+			(project "Chest"
+				(path "/46c350bb-7de4-4e81-aafd-4af55e37aab0"
+					(reference "#PWR054")
+					(unit 1)
+				)
+			)
+		)
+	)
+	(symbol
 		(lib_id "power:GND")
 		(at 59.055 162.56 0)
@@
 	)
 	(symbol
+		(lib_id "power:+3.3V")
+		(at 27.94 114.935 0)
+		(unit 1)
+		(exclude_from_sim no)
+		(in_bom yes)
+		(on_board yes)
+		(dnp no)
+		(fields_autoplaced yes)
+		(property "Reference" "#PWR056"
+			(at 27.94 118.745 0)
+			(effects
+				(font
+					(size 1.27 1.27)
+				)
+				(hide yes)
+			)
+		)
+		(property "Value" "+3V3"
+			(at 27.94 111.3592 0)
+			(effects
+				(font
+					(size 1.27 1.27)
+				)
+			)
+		)
+		(property "Footprint" ""
+			(at 27.94 114.935 0)
+			(effects
+				(font
+					(size 1.27 1.27)
+				)
+				(hide yes)
+			)
+		)
+		(property "Datasheet" ""
+			(at 27.94 114.935 0)
+			(effects
+				(font
+					(size 1.27 1.27)
+				)
+				(hide yes)
+			)
+		)
+		(property "Description" "Power symbol creates a global label with name \"+3.3V\""
+			(at 27.94 114.935 0)
+			(effects
+				(font
+					(size 1.27 1.27)
+				)
+				(hide yes)
+			)
+		)
+		(pin "1"
+		)
+		(instances
+			(project "Chest"
+				(path "/46c350bb-7de4-4e81-aafd-4af55e37aab0"
+					(reference "#PWR056")
+					(unit 1)
+				)
+			)
+		)
+	)
+	(symbol
 		(lib_id "power:GND")
 		(at 66.04 60.96 90)
@@
 	)
 	(symbol
-		(lib_id "power:+3.3V")
-		(at 27.94 114.935 0)
-		(unit 1)
-		(exclude_from_sim no)
-		(in_bom yes)
-		(on_board yes)
-		(dnp no)
-		(property "Reference" "#PWR054"
-			(at 27.94 118.745 0)
-			(effects
-				(font
-					(size 1.27 1.27)
-				)
-				(hide yes)
-			)
-		)
-		(property "Value" "+3.3V"
-			(at 27.94 111.3592 0)
-			(effects
-				(font
-					(size 1.27 1.27)
-				)
-			)
-		)
-		(property "Footprint" ""
-			(at 27.94 114.935 0)
-			(effects
-				(font
-					(size 1.27 1.27)
-				)
-				(hide yes)
-			)
-		)
-		(property "Datasheet" ""
-			(at 27.94 114.935 0)
-			(effects
-				(font
-					(size 1.27 1.27)
-				)
-				(hide yes)
-			)
-		)
-		(property "Description" "Power symbol creates a global label with name \"+3.3V\""
-			(at 27.94 114.935 0)
-			(effects
-				(font
-					(size 1.27 1.27)
-				)
-				(hide yes)
-			)
-		)
-		(pin "1"
-		)
-		(instances
-			(project "Chest"
-				(path "/46c350bb-7de4-4e81-aafd-4af55e37aab0"
-					(reference "#PWR054")
-					(unit 1)
-				)
-			)
-		)
-	)
-	(symbol
 		(lib_id "power:GND")
 		(at 164.465 121.285 180)
@@
 					(unit 1)
 				)
-			)
-		)
-	)
-	(symbol
-		(lib_id "power:+3.3V")
-		(at 34.29 114.935 0)
-		(unit 1)
-		(exclude_from_sim no)
-		(in_bom yes)
-		(on_board yes)
-		(dnp no)
-		(property "Reference" "#PWR056"
-			(at 34.29 118.745 0)
-			(effects
-				(font
-					(size 1.27 1.27)
-				)
-				(hide yes)
-			)
-		)
-		(property "Value" "+3.3V"
-			(at 34.29 111.3592 0)
-			(effects
-				(font
-					(size 1.27 1.27)
-				)
-			)
-		)
-		(property "Footprint" ""
-			(at 34.29 114.935 0)
-			(effects
-				(font
-					(size 1.27 1.27)
-				)
-				(hide yes)
-			)
-		)
-		(property "Datasheet" ""
-			(at 34.29 114.935 0)
-			(effects
-				(font
-					(size 1.27 1.27)
-				)
-				(hide yes)
-			)
-		)
-		(property "Description" "Power symbol creates a global label with name \"+3.3V\""
-			(at 34.29 114.935 0)
-			(effects
-				(font
-					(size 1.27 1.27)
-				)
-				(hide yes)
-			)
-		)
-		(pin "1"
-		)
-		(instances
-			(project "Chest"
-				(path "/46c350bb-7de4-4e81-aafd-4af55e37aab0"
-					(reference "#PWR056")
-					(unit 1)
-				)

Commit message: Tidy
Parts:
- removed V1, V4: ~, RevK:VCUT70N, symbol RevK:VCUT
Other:
- moved on the sheet: C5, C6, C7, C8, D4, D5, D6, D7, J6, J7, J8, J9

Commit message: Tweak tracks
Parts:
- R16: value 210R2 -> 210R; LCSC Part # (none) -> C226891
Changed lines of the file:
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@@
 			)
 		)
-		(property "Value" "210R2"
+		(property "Value" "210R"
 			(at 244.348 76.454 90)
 			(effects
@@
 			(effects
 				(font
+					(size 1.27 1.27)
+				)
+				(hide yes)
+			)
+		)
+		(property "LCSC Part #" "C226891"
+			(at 244.475 78.74 90)
+			(effects
+				(font

Commit message: New render
Parts:
- renumbered C6 to C1, C7 to C2, C8 to C3, C3 to C4, L2 to L1, R9 to R1, R10 to R2, R11 to R3, R1 to R6, U5 to U1
Changed lines of the file:
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@@
 (kicad_sch
-	(version 20231120)
+	(version 20241209)
 	(generator "eeschema")
-	(generator_version "8.0")
+	(generator_version "9.0")
 	(paper "A4")
 	(title_block
@@
 		(on_board yes)
 		(dnp no)
-		(property "Reference" "C6"
+		(property "Reference" "C1"
 			(at 56.515 19.685 0)
 			(effects
@@
 		(on_board yes)
 		(dnp no)
-		(property "Reference" "C8"
+		(property "Reference" "C3"
 			(at 58.928 23.622 90)
 			(effects
@@
 		(on_board yes)
 		(dnp no)
-		(property "Reference" "R11"
+		(property "Reference" "R3"
 			(at 56.515 29.21 0)
 			(effects
@@
 		(dnp no)
 		(fields_autoplaced yes)
-		(property "Reference" "#PWR0105"
+		(property "Reference" "#PWR013"
 			(at 80.01 118.745 0)
 			(effects
@@
 		(on_board yes)
 		(dnp no)
-		(property "Reference" "R9"
+		(property "Reference" "R1"
 			(at 57.785 25.4 0)
 			(effects
@@
 		(dnp no)
 		(fields_autoplaced yes)
-		(property "Reference" "#PWR03"
+		(property "Reference" "#PWR08"
 			(at 62.23 55.88 0)
 			(effects
@@
 		(on_board yes)
 		(dnp no)
-		(property "Reference" "#PWR010"
+		(property "Reference" "#PWR03"
 			(at 34.29 41.91 0)
 			(effects
@@
 		(dnp no)
 		(fields_autoplaced yes)
-		(property "Reference" "#PWR0106"
+		(property "Reference" "#PWR012"
 			(at 80.01 100.965 0)
 			(effects
@@
 		(dnp no)
 		(fields_autoplaced yes)
-		(property "Reference" "#PWR01"
+		(property "Reference" "#PWR09"
 			(at 72.39 60.96 0)
 			(effects
@@
 		(on_board yes)
 		(dnp no)
-		(property "Reference" "R1"
+		(property "Reference" "R6"
 			(at 81.915 100.965 90)
 			(effects
@@
 		(on_board yes)
 		(dnp no)
-		(property "Reference" "L2"
+		(property "Reference" "L1"
 			(at 56.515 31.115 90)
 			(effects
@@
 		(on_board yes)
 		(dnp no)
-		(property "Reference" "U5"
+		(property "Reference" "U1"
 			(at 34.29 19.685 0)
 			(effects
@@
 		(on_board yes)
 		(dnp no)
-		(property "Reference" "C7"
+		(property "Reference" "C2"
 			(at 56.515 21.59 0)
 			(effects
@@
 		(dnp no)
 		(fields_autoplaced yes)
-		(property "Reference" "#PWR09"
+		(property "Reference" "#PWR01"
 			(at 26.67 26.035 0)
 			(effects
@@
 		(dnp no)
 		(fields_autoplaced yes)
-		(property "Reference" "C3"
+		(property "Reference" "C4"
 			(at 82.931 107.7503 0)
 			(effects
@@
 		(on_board yes)
 		(dnp no)
-		(property "Reference" "R10"
+		(property "Reference" "R2"
 			(at 57.658 27.178 90)
 			(effects
@@
 		)
 	)
+	(embedded_fonts no)
 )
