File: PCB/Glove/Glove.kicad_pcb (KiCad board)
At the start: 2 copper layers, 70 x 70 mm, 36 parts, among them J1 JST-PH-SM4-TB, J2 USB-C-Socket-V, J3 Wago, J4 Reset, J5 BTN, J7 TC2030-USB-NL-DS, Q1 CJ2301, Q3 CJ2301, U1 ESP32-S3-MINI-1, U3 TP4054, U4 ME6211C33M5G-N

Commit message: Ready to track
Parts:
- removed D24: ~, RevK:DFN1006-2L
- added R6: 10K, RevK:R_0402, F.Cu at (87.2, 100.0)
- moved J3 17.4 mm to (88.0, 107.0)
- moved J5 17.3 mm to (88.0, 95.0)
- moved D1 17.0 mm to (95.5, 102.0), turned to 90 degrees
- moved R7 16.8 mm to (95.5, 108.9)
- moved R8 16.8 mm to (95.5, 110.7)
- moved R9 16.8 mm to (95.5, 107.0)
- moved D3 16.7 mm to (95.5, 100.1), turned to 90 degrees
- moved R11 14.1 mm to (112.5, 111.5), turned to 0 degrees
- moved R3 12.8 mm to (112.2, 96.2)
- moved C26 11.0 mm to (102.0, 108.5), turned to 180 degrees
- moved R2 10.6 mm to (112.2, 98.2), turned to 90 degrees
- moved J7 9.59 mm to (91.8, 100.0), turned to 0 degrees
- moved R4 6.99 mm to (97.0, 109.5)
- moved R5 6.99 mm to (98.9, 109.5)
- moved D2 4.46 mm to (106.0, 108.5), turned to 180 degrees
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Connections:
- J3 pad 3: VBAT -> +3.3V
- U1 pad 23: unconnected-(U1-GPIO19-Pad23) -> D-
- U1 pad 4: Net-(U1-GPIO0) -> unconnected-(U1-GPIO0-Pad4)
Routing:
- added copper zone on B.Cu, net GND
- added copper zone on F.Cu, net GND
Other:
- board text added: "ironman.revk.uk"
- board text removed: "+"
- board text removed: "2 3 4 5 6 7 8 9 10 11 12 13 14 15"
- board text removed: "5060634238182"
- board text removed: "<"
- board text removed: ">"
- board text removed: "AB"
- board text removed: "C"
- board text removed: "RGB GPSTICK CHARGING GPSRX USB GPSTX SDSS SDMOSI SDSCK SDCD SDMISO ACCSDA ACCSCL PWR"
- board text removed: "S"
- board text removed: "gps.revk.uk"
- board text removed: "⎍"
- board text removed: "⏚"

Commit message: Ready to order
Parts:
- moved R3 12.9 mm to (109.0, 108.8)
- moved R2 10.7 mm to (110.0, 108.8), turned to -90 degrees
- moved C2 9.35 mm to (116.1, 102.0)
- moved D3 8.00 mm to (87.5, 100.0), turned to 180 degrees
- moved J2 4.59 mm to (114.3, 95.2)
- moved R5 4.37 mm to (103.0, 108.0), turned to 90 degrees
- moved D1 3.50 mm to (95.5, 105.5)
- moved R4 3.34 mm to (100.3, 110.0)
- moved R6 1.75 mm to (85.5, 100.0)
- moved C26 1.50 mm to (100.5, 108.5)
- moved R7 1.25 mm to (95.5, 110.2)
- moved R8 1.25 mm to (95.5, 112.0)
- moved R9 1.25 mm to (95.5, 108.2)
- moved C5 1.00 mm to (95.5, 93.0)
- moved R1 1.00 mm to (95.5, 95.0)
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Connections:
- U1 pad 10: USB -> unconnected-(U1-GPIO6-Pad10)
- U1 pad 15: unconnected-(U1-GPIO11-Pad15) -> LED
- U1 pad 21: unconnected-(U1-GPIO17-Pad21) -> CHARGING
- U1 pad 22: unconnected-(U1-GPIO18-Pad22) -> USB
- U1 pad 5: BTN -> unconnected-(U1-GPIO1-Pad5)
- U1 pad 6: RGB -> BTN
- U1 pad 7: CHARGING -> unconnected-(U1-GPIO3-Pad7)
- U1 pad 8: LED -> unconnected-(U1-GPIO4-Pad8)
- U1 pad 9: unconnected-(U1-GPIO5-Pad9) -> RGB
Routing:
- net +3.3V: track 0.00 -> 101.9 mm, vias 0 -> 7
- net GND: track 0.00 -> 95.0 mm, vias 0 -> 31
- net VBUS: track 0.00 -> 61.7 mm, vias 0 -> 6
- net D-: track 0.00 -> 43.7 mm, vias 0 -> 2
- net D+: track 0.00 -> 36.3 mm, vias 0 -> 2
- net VBAT: track 0.00 -> 32.8 mm, vias 0 -> 4
- net Net-(J2-CC2): track 0.00 -> 20.5 mm, vias 0 -> 2
- net Net-(U1-EN): track 0.00 -> 18.7 mm, vias 0 -> 2
- net BTN: track 0.00 -> 18.7 mm
- net RGB: track 0.00 -> 15.7 mm
- net Net-(D2-K): track 0.00 -> 15.5 mm
- net Net-(J2-CC1): track 0.00 -> 15.3 mm, vias 0 -> 2
- net LED: track 0.00 -> 14.6 mm
- net USB: track 0.00 -> 13.5 mm, vias 0 -> 2
- net Net-(J4-Pin_2): track 0.00 -> 11.3 mm, vias 0 -> 1
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- added copper zone on F.Cu, net VBUS
Other:
- board text added: "+"
- board text added: "-"
- board text added: "11"
- board text added: "17 18"
- board text added: "2"
- board text added: "3V3"
- board text added: "5"
- board text added: "BTN"
- board text added: "CHG USB"
- board text added: "LED"
- board text added: "®"
