File: PCB/IronMan/IronMan.kicad_pcb (KiCad board)
At the start: 2 copper layers, 70 x 70 mm, 61 parts, among them J1 Reset, J10 L, J11 R, J12 TF_PUSH, J2 A, J3 B, J4 TC2030-USB-NL-DS, J5 USB-C-Socket-H, J6 1, J7 2, J8 3, J9 4, U1 MD8942, U2 ESP32-S3-MINI-1, U3 L, U4 R, U5 MAX98357A, U6 MAX98357A

Commit message: Tweak - 5V MAX
Parts:
- moved C12 2.02 mm to (111.8, 85.1), turned to 180 degrees
- moved D3 1.57 mm to (90.8, 95.0)
- moved D4 0.89 mm to (89.2, 96.0)
- moved C11 0.71 mm to (86.5, 89.5), turned to -90 degrees
- moved C13 0.71 mm to (85.5, 89.5), turned to -90 degrees
- moved C10 0.57 mm to (110.6, 83.5)
- moved C14 0.50 mm to (111.8, 85.9)
- moved U6 0.50 mm to (113.0, 87.5)
Connections:
- C11 pad 1: +3V3 -> DC
- C12 pad 1: +3V3 -> DC
- C13 pad 1: +3V3 -> DC
- C14 pad 1: +3V3 -> DC
- U5 pad A2: +3V3 -> DC
- U6 pad A2: +3V3 -> DC
Routing:
- net DC: track 152.6 -> 194.1 mm, vias 5 -> 11
- net +3V3: track 209.1 -> 204.8 mm
- net GND: track 111.0 -> 107.0 mm, vias 39 -> 45
- net LED0: track 1.30 -> 2.85 mm
- net LED1: track 19.6 -> 21.1 mm, vias 0 -> 1
- net SPKSD: track 46.1 -> 45.2 mm
- net Net-(J11-Pin_2): track 14.8 -> 15.5 mm, vias 0 -> 1
- net MICWS: track 44.5 -> 45.0 mm
- net Net-(U6-~{SD_MODE}): track 4.21 -> 3.71 mm
- net SPKWS: track 46.5 -> 46.0 mm
- net SPKSCK: track 45.2 -> 44.7 mm
- net Net-(J11-Pin_1): vias 0 -> 1
- net BTNB: vias 2 -> 3
- net Net-(J10-Pin_2): vias 0 -> 1
- net Net-(J10-Pin_1): vias 0 -> 1
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Other:
- board text added: "5V"
