File: PCB/IronMan/IronMan.kicad_pcb (KiCad board)
At the start: 2 copper layers, 70 x 70 mm, 61 parts, among them J1 Reset, J10 L, J11 R, J12 TF_PUSH, J2 A, J3 B, J4 TC2030-USB-NL-DS, J5 USB-C-Socket-H, J6 1, J7 2, J8 3, J9 4, U1 MD8942, U2 ESP32-S3-MINI-1, U3 L, U4 R, U5 MAX98357A, U6 MAX98357A

Commit message: Pos files
Parts:
- U3, U4: footprint RevK:ICS43434_MEMS_Mic_Open -> RevK:ICS43434_MEMS_Mic

Commit message: manual
Connections:
- J4 pad 2: DC -> D-
- J4 pad 6: GND -> D-
Routing:
- net D+: track 46.2 -> 36.9 mm
- net D-: track 35.7 -> 38.8 mm
- net GND: track 107.0 -> 107.7 mm, vias 45 -> 46

Commit message: Image eupdates
Parts:
- C5, C6, C7, C8: value C_Polarized -> 470uF
- J4: moved to B.Cu
- moved J4 2.09 mm to (88.5, 101.5), turned to 0 degrees
- moved D7 1.00 mm to (111.0, 102.0)
Connections:
- net DC renamed +5V
- net SPKSCK renamed SPKBSCK
- net SPKSD renamed SPKDATA
- net SPKWS renamed SPKLRC
Routing:
- net +5V: track 193.7 -> 182.2 mm
- net LED3: track 36.6 -> 31.0 mm, vias 3 -> 1
- net MICSD: track 49.6 -> 44.3 mm
- net GND: track 107.7 -> 103.6 mm
- net D-: track 38.8 -> 35.4 mm, vias 3 -> 2
- net MICWS: track 45.0 -> 43.0 mm
- net +3V3: track 204.8 -> 206.5 mm
- net D+: track 36.9 -> 36.7 mm, vias 3 -> 2
Other:
- board text added: "A"
- board text added: "LRC BCLK DATA PWR"
- board text added: "TC2030"
- board text added: "U"
- board text added: "hiwtsi.uk"
- board text added: "ironman.revk.uk"
- board text removed: "WS SCK SD PWR"
- board text removed: "ironman.revk.uk hiwtsi.uk"
