File: PCB/IronMan/IronMan.kicad_sch (KiCad schematic)
At the start: 61 parts, among them J1 Reset, J10 L, J11 R, J12 TF_PUSH, J2 A, J3 B, J4 TC2030-USB-NL-DS, J5 USB-C-Socket-H, J6 1, J7 2, J8 3, J9 4, U1 MD8942, U2 ESP32-S3-MINI-1, U3 L, U4 R, U5 MAX98357A, U6 MAX98357A

Commit message: Tweak - 5V MAX
Connections:
- net +3V3: no longer C11.1, C12.1, C13.1, C14.1, U5.A2 (VDD), U6.A2 (VDD)
- net DC: now also C11.1, C12.1, C13.1, C14.1, U5.A2 (VDD), U6.A2 (VDD)
Other:
- moved on the sheet: C13, C14

Commit message: Library update
Parts:
- U1: Rotation Offset (none) -> 180
Changed lines of the file:
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@@
+			)
+		)
+		(property "Rotation Offset" "180"
+			(at 34.29 26.035 0)
+			(effects
+				(font
+					(size 1.27 1.27)
+				)
+				(hide yes)
 			)
 		)

Commit message: Pos files
Parts:
- D1, D2, D4, D5, D6, D7: MPN (none) -> C5137770
- D3: MPN (none) -> C5349953
- J12: JLCPCB Position Offset 0,3.075 -> (none); LCSC Part # C393941 -> (none); MPN (none) -> C393941; Position Offset (none) -> 0,0.15
- J5: LCSC Part # C709357 -> (none); MPN (none) -> C709357; Position Offset (none) -> 0,0.715
- U1: MPN (none) -> C2684786
- U2: LCSC Part # C3013941 -> (none); MPN (none) -> C3013941
- U3, U4: footprint RevK:ICS43434_MEMS_Mic_Open -> RevK:ICS43434_MEMS_Mic; LCSC Part # C5656610 -> (none); MPN (none) -> C5656610
- U5, U6: MPN (none) -> C2682619
Changed lines of the file:
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@@
 			)
 		)
-		(property "Description" ""
+		(property "Description" "Polarized capacitor"
 			(at 137.16 156.21 0)
 			(effects
@@
 			)
 		)
+		(property "MPN" "C5137770"
+			(at 105.41 137.795 0)
+			(effects
+				(font
+					(size 1.27 1.27)
+				)
+				(hide yes)
+			)
+		)
 		(pin "2"
 		)
@@
 			)
 		)
-		(property "Description" ""
+		(property "Description" "Resistor"
 			(at 210.185 129.54 0)
 			(effects
@@
 			)
 		)
-		(property "Description" ""
+		(property "Description" "Resistor"
 			(at 213.995 129.54 0)
 			(effects
@@
 			)
 		)
-		(property "Description" ""
+		(property "Description" "Unpolarized capacitor"
 			(at 187.325 63.5 0)
 			(effects
@@
 			)
 		)
-		(property "Description" ""
+		(property "Description" "ESP32S3"
 			(at 50.8 77.47 0)
 			(effects
@@
 			)
 		)
-		(property "LCSC Part #" "C3013941"
+		(property "MPN" "C3013941"
 			(at 50.8 109.855 0)
 			(effects
@@
 			)
 		)
-		(property "Description" ""
+		(property "Description" "Unpolarized capacitor"
 			(at 272.415 78.105 0)
 			(effects
@@
 			)
 		)
-		(property "Description" ""
+		(property "Description" "Power symbol creates a global label with name \"GND\" , ground"
 			(at 277.495 160.02 0)
 			(effects
@@
 			)
 		)
-		(property "Description" ""
+		(property "Description" "Power symbol creates a global label with name \"GND\" , ground"
 			(at 227.965 90.17 0)
 			(effects
@@
 			)
 		)
-		(property "Description" ""
+		(property "Description" "Resistor"
 			(at 233.045 129.54 0)
 			(effects
@@
 			)
 		)
-		(property "Description" ""
+		(property "Description" "Unpolarized capacitor"
 			(at 265.43 35.56 0)
 			(effects
@@
 			)
 		)
-		(property "Description" ""
+		(property "Description" "Power symbol creates a global label with name \"GND\" , ground"
 			(at 240.665 81.28 0)
 			(effects
@@
 			)
 		)
-		(property "Footprint" "RevK:ICS43434_MEMS_Mic_Open"
+		(property "Footprint" "RevK:ICS43434_MEMS_Mic"
 			(at 162.306 45.085 0)
 			(effects
@@
 			)
 		)
-		(property "LCSC Part #" "C5656610"
+		(property "MPN" "C5656610"
 			(at 168.91 72.263 0)
 			(effects
@@
 			)
 		)
-		(property "Description" ""
+		(property "Description" "Power symbol creates a global label with name \"GND\" , ground"
 			(at 227.965 48.26 0)
 			(effects
@@
 			)
 		)
-		(property "Footprint" "RevK:ICS43434_MEMS_Mic_Open"
+		(property "Footprint" "RevK:ICS43434_MEMS_Mic"
 			(at 162.306 13.97 0)
 			(effects
@@
 			)
 		)
-		(property "LCSC Part #" "C5656610"
+		(property "MPN" "C5656610"
 			(at 168.91 41.148 0)
 			(effects
@@
 			)
 		)
+		(property "MPN" "C5137770"
+			(at 140.335 166.37 0)
+			(effects
+				(font
+					(size 1.27 1.27)
+				)
+				(hide yes)
+			)
+		)
 		(pin "2"
 		)
@@
 			)
 		)
-		(property "Datasheet" " ~"
+		(property "Datasheet" "~"
 			(at 91.44 27.305 0)
 			(effects
@@
 			)
 		)
+		(property "MPN" "C5137770"
+			(at 62.23 158.75 0)
+			(effects
+				(font
+					(size 1.27 1.27)
+				)
+				(hide yes)
+			)
+		)
 		(pin "2"
 		)
@@
 			)
 		)
+		(property "MPN" "C5137770"
+			(at 105.41 166.37 0)
+			(effects
+				(font
+					(size 1.27 1.27)
+				)
+				(hide yes)
+			)
+		)
 		(pin "2"
 		)
@@
 			)
 		)
-		(property "Description" ""
+		(property "Description" "Unpolarized capacitor"
 			(at 271.78 35.56 0)
 			(effects
@@
 			)
 		)
-		(property "Description" ""
+		(property "Description" "Micro SD Card Socket"
 			(at 257.175 144.78 0)
 			(effects
@@
 			)
 		)
-		(property "LCSC Part #" "C393941"
+		(property "MPN" "C393941"
 			(at 257.175 144.78 0)
 			(effects
@@
 			)
 		)
-		(property "JLCPCB Position Offset" "0,3.075"
+		(property "Position Offset" "0,0.15"
 			(at 257.175 144.78 0)
 			(effects
@@
 			)
 		)
-		(property "Description" ""
+		(property "Description" "Power symbol creates a global label with name \"GND\" , ground"
 			(at 240.665 39.37 0)
 			(effects
@@
 			)
 		)
-		(property "Description" ""
+		(property "Description" "Resistor"
 			(at 229.235 129.54 0)
 			(effects
@@
 			)
 		)
-		(property "LCSC Part #" "C709357"
+		(property "MPN" "C709357"
+			(at 92.71 58.42 0)
+			(effects
+				(font
+					(size 1.27 1.27)
+				)
+				(hide yes)
+			)
+		)
+		(property "Position Offset" "0,0.715"
 			(at 92.71 58.42 0)
 			(effects
@@
 	)
 	(symbol
+		(lib_name "MAX98357A_1")
 		(lib_id "RevK:MAX98357A")
 		(at 227.965 35.56 0)
@@
 			)
 		)
-		(property "LCSC Part #" ""
+		(property "MPN" "C2682619"
 			(at 227.965 35.56 0)
 			(effects
@@
 					(size 1.27 1.27)
 				)
+				(hide yes)
 			)
 		)
@@
 			)
 		)
-		(property "Description" ""
+		(property "Description" "Polarized capacitor"
 			(at 102.235 156.21 0)
 			(effects
@@
 			)
 		)
-		(property "LCSC Part #" ""
+		(property "MPN" "C2682619"
 			(at 227.965 77.47 0)
 			(effects
@@
 					(size 1.27 1.27)
 				)
+				(hide yes)
 			)
 		)
@@
 			)
 		)
-		(property "Description" ""
+		(property "Description" "Resistor"
 			(at 221.615 129.54 0)
 			(effects
@@
 			)
 		)
+		(property "MPN" "C5137770"
+			(at 140.335 137.795 0)
+			(effects
+				(font
+					(size 1.27 1.27)
+				)
+				(hide yes)
+			)
+		)
 		(pin "2"
 		)
@@
 			)
 		)
+		(property "MPN" "C5349953"
+			(at 103.505 87.63 0)
+			(effects
+				(font
+					(size 1 1)
+				)
+				(justify left top)
+				(hide yes)
+			)
+		)
 		(pin "1"
 		)
@@
 			)
 		)
-		(property "Description" ""
+		(property "Description" "Unpolarized capacitor"
 			(at 34.29 118.745 0)
 			(effects
@@
 			)
 		)
-		(property "Description" ""
+		(property "Description" "Polarized capacitor"
 			(at 102.235 127.635 0)
 			(effects
@@
 			)
 		)
+		(property "MPN" "C2684786"
+			(at 34.29 52.705 0)
+			(effects
+				(font
+					(size 1.27 1.27)
+				)
+				(hide yes)
+			)
+		)
 		(pin "1"
 		)
@@
 			)
 		)
-		(property "Description" ""
+		(property "Description" "Polarized capacitor"
 			(at 137.16 127.635 0)
 			(effects
@@
 			)
 		)
-		(property "Description" ""
+		(property "Description" "Unpolarized capacitor"
 			(at 187.325 32.385 0)
 			(effects
@@
 			)
 		)
-		(property "Description" ""
+		(property "Description" "Resistor"
 			(at 225.425 129.54 0)
 			(effects
@@
 			)
 		)
+		(property "MPN" "C5137770"
+			(at 62.23 134.62 0)
+			(effects
+				(font
+					(size 1.27 1.27)
+				)
+				(hide yes)
+			)
+		)
 		(pin "2"
 		)
@@
 			)
 		)
-		(property "Description" ""
+		(property "Description" "Unpolarized capacitor"
 			(at 27.94 118.745 0)
 			(effects
@@
 			)
 		)
-		(property "Description" ""
+		(property "Description" "Resistor"
 			(at 217.805 129.54 0)
 			(effects
@@
 			)
 		)
-		(property "Description" ""
+		(property "Description" "Unpolarized capacitor"
 			(at 266.065 78.105 0)
 			(effects

Commit message: PCB Update
Parts:
- C1: LCSC Part # C194427 -> (none); MPN (none) -> C194427
- C11, C12: LCSC Part # C15525 -> (none); MPN (none) -> C15525
- C2: LCSC Part # C1691 -> (none); MPN (none) -> C1691
- C5, C6, C7, C8: JLCPCB Rotation Offset 180 -> (none); LCSC Part # C106188 -> (none); MPN (none) -> C106188
- D1, D2, D4, D5, D6, D7: LCSC Part # C5137770 -> (none)
- D3: LCSC Part # C5349953 -> (none)
- J10, J11, J2, J3: LCSC Part # C2765055 -> (none); MPN (none) -> C2765055
- J12: Position Offset 0,0.15 -> (none)
- J5: Position Offset 0,0.715 -> (none)
- J6, J7, J8, J9: LCSC Part # C2765056 -> (none); MPN (none) -> C2765056
- R16: LCSC Part # C226891 -> (none); MPN (none) -> C226891
- U1: LCSC Part # C2684786 -> (none); MPN C2684786 -> (none); Rotation Offset 180 -> (none)
Changed lines of the file:
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@@
 			)
 		)
-		(property "LCSC Part #" "C194427"
+		(property "MPN" "C194427"
 			(at 55.245 19.685 0)
 			(effects
@@
 			)
 		)
-		(property "LCSC Part #" "C106188"
-			(at 137.16 156.21 0)
-			(effects
-				(font
-					(size 1.27 1.27)
-				)
-				(hide yes)
-			)
-		)
-		(property "JLCPCB Rotation Offset" "180"
+		(property "MPN" "C106188"
 			(at 137.16 156.21 0)
 			(effects
@@
 			)
 		)
-		(property "LCSC Part #" "C5137770"
+		(property "MPN" "C5137770"
 			(at 105.41 137.795 0)
 			(effects
@@
 			)
 		)
-		(property "LCSC Part #" "C15525"
+		(property "MPN" "C15525"
 			(at 265.43 35.56 0)
 			(effects
@@
 			)
 		)
-		(property "LCSC Part #" "C2765055"
+		(property "MPN" "C2765055"
 			(at 81.28 133.35 0)
 			(effects
@@
 			)
 		)
-		(property "LCSC Part #" "C5137770"
+		(property "MPN" "C5137770"
 			(at 140.335 166.37 0)
 			(effects
@@
 			)
 		)
-		(property "LCSC Part #" "C5137770"
+		(property "MPN" "C5137770"
 			(at 62.23 158.75 0)
 			(effects
@@
 			)
 		)
-		(property "LCSC Part #" "C5137770"
+		(property "MPN" "C5137770"
 			(at 105.41 166.37 0)
 			(effects
@@
 			)
 		)
-		(property "Position Offset" "0,0.15"
-			(at 257.175 144.78 0)
-			(effects
-				(font
-					(size 1.27 1.27)
-				)
-				(hide yes)
-			)
-		)
 		(pin "1"
 		)
@@
 			)
 		)
-		(property "Position Offset" "0,0.715"
-			(at 92.71 58.42 0)
-			(effects
-				(font
-					(size 1.27 1.27)
-				)
-				(hide yes)
-			)
-		)
 		(pin "A1"
 		)
@@
 			)
 		)
-		(property "LCSC Part #" "C106188"
-			(at 102.235 156.21 0)
-			(effects
-				(font
-					(size 1.27 1.27)
-				)
-				(hide yes)
-			)
-		)
-		(property "JLCPCB Rotation Offset" "180"
+		(property "MPN" "C106188"
 			(at 102.235 156.21 0)
 			(effects
@@
 			)
 		)
-		(property "LCSC Part #" "C2765056"
+		(property "MPN" "C2765056"
 			(at 156.21 133.985 0)
 			(effects
@@
 			)
 		)
-		(property "LCSC Part #" "C2765056"
+		(property "MPN" "C2765056"
 			(at 156.21 162.56 0)
 			(effects
@@
 			)
 		)
-		(property "LCSC Part #" "C2765056"
+		(property "MPN" "C2765056"
 			(at 121.285 133.985 0)
 			(effects
@@
 			)
 		)
-		(property "LCSC Part #" "C5137770"
+		(property "MPN" "C5137770"
 			(at 140.335 137.795 0)
 			(effects
@@
 			)
 		)
-		(property "LCSC Part #" "C2765055"
+		(property "MPN" "C2765055"
 			(at 245.745 30.48 0)
 			(effects
@@
 			)
 		)
-		(property "LCSC Part #" "C2765055"
+		(property "MPN" "C2765055"
 			(at 81.28 157.48 0)
 			(effects
@@
 			)
 		)
-		(property "LCSC Part #" "C5349953"
+		(property "MPN" "C5349953"
 			(at 103.505 87.63 0)
 			(effects
@@
 			)
 		)
-		(property "LCSC Part #" "C2765056"
+		(property "MPN" "C2765056"
 			(at 121.285 162.56 0)
 			(effects
@@
 			)
 		)
-		(property "LCSC Part #" "C106188"
-			(at 102.235 127.635 0)
-			(effects
-				(font
-					(size 1.27 1.27)
-				)
-				(hide yes)
-			)
-		)
-		(property "JLCPCB Rotation Offset" "180"
+		(property "MPN" "C106188"
 			(at 102.235 127.635 0)
 			(effects
@@
 			)
 		)
-		(property "Description" ""
+		(property "Description" "Regulator and associated components."
 			(at 34.29 26.035 0)
 			(effects
@@
 			)
 		)
-		(property "LCSC Part #" "C2684786"
-			(at 34.29 52.705 0)
-			(effects
-				(font
-					(size 1.27 1.27)
-				)
-				(hide yes)
-			)
-		)
-		(property "Rotation Offset" "180"
-			(at 34.29 26.035 0)
-			(effects
-				(font
-					(size 1.27 1.27)
-				)
-				(hide yes)
-			)
-		)
-		(property "MPN" "C2684786"
-			(at 34.29 52.705 0)
-			(effects
-				(font
-					(size 1.27 1.27)
-				)
-				(hide yes)
-			)
-		)
 		(pin "1"
 		)
@@
 			)
 		)
-		(property "LCSC Part #" "C106188"
-			(at 137.16 127.635 0)
-			(effects
-				(font
-					(size 1.27 1.27)
-				)
-				(hide yes)
-			)
-		)
-		(property "JLCPCB Rotation Offset" "180"
+		(property "MPN" "C106188"
 			(at 137.16 127.635 0)
 			(effects
@@
 			)
 		)
-		(property "LCSC Part #" "C2765055"
+		(property "MPN" "C2765055"
 			(at 245.745 72.39 0)
 			(effects
@@
 			)
 		)
-		(property "LCSC Part #" "C1691"
+		(property "MPN" "C1691"
 			(at 55.245 21.59 0)
 			(effects
@@
 			)
 		)
-		(property "LCSC Part #" "C226891"
+		(property "MPN" "C226891"
 			(at 244.475 78.74 90)
 			(effects
@@
 			)
 		)
-		(property "LCSC Part #" "C5137770"
+		(property "MPN" "C5137770"
 			(at 62.23 134.62 0)
 			(effects
@@
 			)
 		)
-		(property "LCSC Part #" "C15525"
+		(property "MPN" "C15525"
 			(at 266.065 78.105 0)
 			(effects

Commit message: manual
Connections:
- net D-: now also J4.2 (NC), J4.6 (NC)
- net DC: no longer J4.2 (VBUS)
- net GND: no longer J4.6 (GND)

Commit message: Image eupdates
Parts:
- C5, C6, C7, C8: value C_Polarized -> 470uF
- U1: MPN (none) -> C2684786
Connections:
- net DC renamed +5V
- net SPKSCK renamed SPKBSCK
- net SPKSD renamed SPKDATA
- net SPKWS renamed SPKLRC
